Commit message: Fixed Gazebo Physics

File: urdf/junior.urdf (robot description, URDF)
Before this commit: robot Junior, 10 links, 9 joints
Links:
- link BackBumper: geometry collision mesh filename=file://$(find junior_model)/meshes/robitBackBumper.stl; visual mesh filename=file://$(find junior_model)/meshes/robitBackBumper.stl
- link Chassis: geometry collision mesh filename=file://$(find junior_model)/meshes/robitChassis.stl; visual mesh filename=file://$(find junior_model)/meshes/robitChassis.stl
- link FrontBumper: geometry collision mesh filename=file://$(find junior_model)/meshes/robitFrontBumper.stl; visual mesh filename=file://$(find junior_model)/meshes/robitFrontBumper.stl
- link FrontLidar: geometry collision mesh filename=file://$(find junior_model)/meshes/robitFrontLidarCase.stl; visual mesh filename=file://$(find junior_model)/meshes/robitFrontLidarCase.stl
- link FrontLidarGlass: geometry collision mesh filename=file://$(find junior_model)/meshes/robitFrontLidarGlass.stl; visual mesh filename=file://$(find junior_model)/meshes/robitFrontLidarGlass.stl
- link WheelLeftBack: geometry collision mesh filename=file://$(find junior_model)/meshes/robitWheel.stl; visual mesh filename=file://$(find junior_model)/meshes/robitWheel.stl
- link WheelLeftFront: geometry collision mesh filename=file://$(find junior_model)/meshes/robitWheel.stl; visual mesh filename=file://$(find junior_model)/meshes/robitWheel.stl
- link WheelRightBack: geometry collision mesh filename=file://$(find junior_model)/meshes/robitWheel.stl; visual mesh filename=file://$(find junior_model)/meshes/robitWheel.stl
- link WheelRightFront: geometry collision mesh filename=file://$(find junior_model)/meshes/robitWheel.stl; visual mesh filename=file://$(find junior_model)/meshes/robitWheel.stl
- link base_link: mass 0.01 -> None

Commit message: Fixed Physics

File: urdf/junior.urdf (robot description, URDF)
Before this commit: robot Junior, 10 links, 9 joints
Links:
- link BackBumper: mass 0.01 -> 1
- link Chassis: mass 0.01 -> 1
- link FrontBumper: mass 0.01 -> 1
- link FrontLidar: mass 0.01 -> 1
- link FrontLidarGlass: mass 0.01 -> 1
- link WheelLeftBack: mass 0.01 -> 1
- link WheelLeftFront: mass 0.01 -> 1
- link WheelRightBack: mass 0.01 -> 1
- link WheelRightFront: mass 0.01 -> 1
Joints:
- joint ChassisJoint: origin xyz=1 0 0.23 -> xyz=1 0 1

Commit message: Fixed Physics Again

File: urdf/junior.urdf (robot description, URDF)
Before this commit: robot Junior, 10 links, 9 joints
Joints:
- joint ChassisJoint: origin xyz=1 0 1 -> xyz=1 0 0.23

Commit message: Fixed Physics Again

File: urdf/junior.urdf (robot description, URDF)
Before this commit: robot Junior, 10 links, 9 joints
Joints:
- joint ChassisJoint: origin xyz=1 0 0.23 -> xyz=0 0 0.23
